File: PCB/plugboard.sch (KiCad schematic (older format))
At the start: 95 parts, among them J1 1/4\" Jack, J10 Conn_01x19_Male_0, J11 Conn_01x19_Male_0, J2 1/4\" Jack, J3 1/4\" Jack, J4 1/4\" Jack, J5 1/4\" Jack, J6 1/4\" Jack, J7 1/4\" Jack, J8 1/4\" Jack, J9 1/4\" Jack, P1 CONN_02X03, P2 CONN_02X03, U1 ADG732

Commit message: add .gitignore
Parts:
- R15, R16, R17, R18, R19, R20, R21, R22, R23, R24, R26, R27, R28, R29, R30, R31, R34, R35, R36, R37, R38, R39, R41, R42, R43, R44, R45, R46, R47, R48, R49, R50, R51, R52, R55, R56, R57, R58, R59, R60, R62, R63, R64, R65, R66, R67, R69, R70, R71, R72, R73, R74: footprint (none) -> footprints:R_0805_OEM

Commit message: Add footprints library
Parts:
- P1, P2: footprint footprints:Pin_Header_Straight_2x03 -> enigmaprints:Pin_Header_Straight_2x03
- R1, R10, R11, R12, R13, R14, R15, R16, R17, R18, R19, R2, R20, R21, R22, R23, R24, R25, R26, R27, R28, R29, R3, R30, R31, R32, R33, R34, R35, R36, R37, R38, R39, R4, R40, R41, R42, R43, R44, R45, R46, R47, R48, R49, R5, R50, R51, R52, R53, R54, R55, R56, R57, R58, R59, R6, R60, R61, R62, R63, R64, R65, R66, R67, R68, R69, R7, R70, R71, R72, R73, R74, R75, R76, R77, R78, R79, R8, R80, R9: footprint footprints:R_0805_OEM -> enigmaprints:R_0805_OEM

Commit message: added pull down resistors
Parts:
- added R? (x26): R_10K, enigmaprints:R_0805_OEM, symbol formula:R_10K
- J1, J2, J3, J4, J5, J6, J7, J8, J9: symbol library:audio_jack -> plugboard-rescue:audio_jack-library
Connections:
- wire segments 110 -> 162
Other:
- moved on the sheet: R15, R16, R17, R18, R19, R20, R21, R22, R23, R24, R26, R27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
