File: PCB/plugboard.sch (KiCad schematic (older format))
At the start: 95 parts, among them J1 1/4\" Jack, J10 Conn_01x19_Male_0, J11 Conn_01x19_Male_0, J2 1/4\" Jack, J3 1/4\" Jack, J4 1/4\" Jack, J5 1/4\" Jack, J6 1/4\" Jack, J7 1/4\" Jack, J8 1/4\" Jack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

Commit message: Add jack and bar parts
Parts:
- J1, J2, J3, J4, J5, J6, J7, J8, J9: footprint footprints:Through Hole -> enigmaprints:jack_hole
- J10, J11: footprint (none) -> enigmaprints:sidebar
Changed lines of the file:
@@
 F 0 "J3" H 4954 5042 50  0000 C CNN
 F 1 "1/4\" Jack" H 4954 4951 50  0000 C CNN
-F 2 "footprints:Through Hole" H 5550 3950 50  0001 C CIN
+F 2 "enigmaprints:jack_hole" H 5550 3950 50  0001 C CIN
 F 3 "http://www.switchcraft.com/Drawings/110x-m110x_series_cd.pdf" H 3350 5880 50  0001 C CNN
 F 4 "112BX" H 4300 4050 60  0001 C CNN "MPN"
@@
 F 0 "J6" H 6304 5042 50  0000 C CNN
 F 1 "1/4\" Jack" H 6304 4951 50  0000 C CNN
-F 2 "footprints:Through Hole" H 6900 3950 50  0001 C CIN
+F 2 "enigmaprints:jack_hole" H 6900 3950 50  0001 C CIN
 F 3 "http://www.switchcraft.com/Drawings/110x-m110x_series_cd.pdf" H 4700 5880 50  0001 C CNN
 F 4 "112BX" H 5650 4050 60  0001 C CNN "MPN"
@@
 F 0 "J8" H 7654 3992 50  0000 C CNN
 F 1 "1/4\" Jack" H 7654 3901 50  0000 C CNN
-F 2 "footprints:Through Hole" H 8250 2900 50  0001 C CIN
+F 2 "enigmaprints:jack_hole" H 8250 2900 50  0001 C CIN
 F 3 "http://www.switchcraft.com/Drawings/110x-m110x_series_cd.pdf" H 6050 4830 50  0001 C CNN
 F 4 "112BX" H 7000 3000 60  0001 C CNN "MPN"
@@
 F 0 "J4" H 6304 2892 50  0000 C CNN
 F 1 "1/4\" Jack" H 6304 2801 50  0000 C CNN
-F 2 "footprints:Through Hole" H 6900 1800 50  0001 C CIN
+F 2 "enigmaprints:jack_hole" H 6900 1800 50  0001 C CIN
 F 3 "http://www.switchcraft.com/Drawings/110x-m110x_series_cd.pdf" H 4700 3730 50  0001 C CNN
 F 4 "112BX" H 5650 1900 60  0001 C CNN "MPN"
@@
 F 0 "J2" H 4954 3992 50  0000 C CNN
 F 1 "1/4\" Jack" H 4954 3901 50  0000 C CNN
-F 2 "footprints:Through Hole" H 5550 2900 50  0001 C CIN
+F 2 "enigmaprints:jack_hole" H 5550 2900 50  0001 C CIN
 F 3 "http://www.switchcraft.com/Drawings/110x-m110x_series_cd.pdf" H 3350 4830 50  0001 C CNN
 F 4 "112BX" H 4300 3000 60  0001 C CNN "MPN"
@@
 F 0 "J5" H 6304 3992 50  0000 C CNN
 F 1 "1/4\" Jack" H 6304 3901 50  0000 C CNN
-F 2 "footprints:Through Hole" H 6900 2900 50  0001 C CIN
+F 2 "enigmaprints:jack_hole" H 6900 2900 50  0001 C CIN
 F 3 "http://www.switchcraft.com/Drawings/110x-m110x_series_cd.pdf" H 4700 4830 50  0001 C CNN
 F 4 "112BX" H 5650 3000 60  0001 C CNN "MPN"
@@
 F 0 "J9" H 7654 5092 50  0000 C CNN
 F 1 "1/4\" Jack" H 7654 5001 50  0000 C CNN
-F 2 "footprints:Through Hole" H 8250 4000 50  0001 C CIN
+F 2 "enigmaprints:jack_hole" H 8250 4000 50  0001 C CIN
 F 3 "http://www.switchcraft.com/Drawings/110x-m110x_series_cd.pdf" H 6050 5930 50  0001 C CNN
 F 4 "112BX" H 7000 4100 60  0001 C CNN "MPN"
@@
 F 0 "J1" H 4954 2892 50  0000 C CNN
 F 1 "1/4\" Jack" H 4954 2801 50  0000 C CNN
-F 2 "footprints:Through Hole" H 5550 1800 50  0001 C CIN
+F 2 "enigmaprints:jack_hole" H 5550 1800 50  0001 C CIN
 F 3 "http://www.switchcraft.com/Drawings/110x-m110x_series_cd.pdf" H 3350 3730 50  0001 C CNN
 F 4 "112BX" H 4300 1900 60  0001 C CNN "MPN"
@@
 F 0 "J7" H 7654 2892 50  0000 C CNN
 F 1 "1/4\" Jack" H 7654 2801 50  0000 C CNN
-F 2 "footprints:Through Hole" H 8250 1800 50  0001 C CIN
+F 2 "enigmaprints:jack_hole" H 8250 1800 50  0001 C CIN
 F 3 "http://www.switchcraft.com/Drawings/110x-m110x_series_cd.pdf" H 6050 3730 50  0001 C CNN
 F 4 "112BX" H 7000 1900 60  0001 C CNN "MPN"
@@
 F 0 "J10" H 10056 3778 50  0000 C CNN
 F 1 "Conn_01x19_Male_0" H 10056 3687 50  0000 C CNN
-F 2 "" H 9950 2700 50  0001 C CNN
+F 2 "enigmaprints:sidebar" H 9950 2700 50  0001 C CNN
 F 3 "~" H 9950 2700 50  0001 C CNN
 	1    9950 2700
@@
 F 0 "J11" H 10056 6278 50  0000 C CNN
 F 1 "Conn_01x19_Male_0" H 10056 6187 50  0000 C CNN
-F 2 "" H 9950 5200 50  0001 C CNN
+F 2 "enigmaprints:sidebar" H 9950 5200 50  0001 C CNN
 F 3 "~" H 9950 5200 50  0001 C CNN
 	1    9950 5200
