File: PCB/plugboard.sch (KiCad schematic (older format))
At the start: 96 parts, among them J1 1/4\" Jack, J10 1/4\" Jack, J11 Conn_01x19_Male_0, J2 1/4\" Jack, J3 1/4\" Jack, J4 1/4\" Jack, J5 1/4\" Jack, J6 1/4\" Jack, J7 Conn_01x19_Male_0, J8 1/4\" Jack, J9 1/4\" Jack, P1 CONN_02X03, P2 CONN_02X03, U1 ADG732

Commit message: Finish first draft layout
Connections:
- net SA: now also U1.11 (S2); no longer U1.36 (S28)
- net SB: now also U1.35 (S27); no longer U1.11 (S2)
- net SC: now also U1.6 (S7); no longer U1.31 (S23)
- net SD: now also U1.3 (S10); no longer U1.28 (S20)
- net SE: now also U1.28 (S20); no longer U1.4 (S9)
- net SG: now also U1.32 (S24); no longer U1.8 (S5)
- net SH: now also U1.4 (S9); no longer U1.29 (S21)
- net SI: now also U1.10 (S3); no longer U1.35 (S27)
- net SJ: now also U1.12 (S1); no longer U1.38 (S30)
- net SK: now also U1.33 (S25); no longer U1.9 (S4)
- net SL: now also U1.36 (S28); no longer U1.12 (S1)
- net SM: now also U1.27 (S19); no longer U1.3 (S10)
- net SN: now also U1.7 (S6); no longer U1.32 (S24)
- net SO: now also U1.30 (S22); no longer U1.6 (S7)
- net SP: now also U1.5 (S8); no longer U1.30 (S22)
- net SQ: now also U1.48 (S13); no longer U1.25 (S17)
- net SR: now also U1.1 (S12); no longer U1.26 (S18)
- net SS: now also U1.31 (S23); no longer U1.7 (S6)
- net ST: now also U1.9 (S4); no longer U1.34 (S26)
- net SU: now also U1.2 (S11); no longer U1.27 (S19)
- net SV: now also U1.26 (S18); no longer U1.2 (S11)
- net SW: now also U1.8 (S5); no longer U1.33 (S25)
- net SX: now also U1.34 (S26); no longer U1.10 (S3)
- net SY: now also U1.25 (S17); no longer U1.1 (S12)
- net SZ: now also U1.29 (S21); no longer U1.5 (S8)
Changed lines of the file:
@@
 Text Label 6550 2950 3    50   ~ 0
 SW
+Text Label 4050 6150 0    50   ~ 0
+SY
+Text Label 4050 4800 0    50   ~ 0
+SX
+Text Label 1500 4800 2    50   ~ 0
+SD
 Text Label 1500 4500 2    50   ~ 0
-SY
+SR
+Text Label 1500 5250 2    50   ~ 0
+SC
+Text Label 4050 6000 0    50   ~ 0
+SV
+Text Label 4050 4650 0    50   ~ 0
+SB
+Text Label 1500 4950 2    50   ~ 0
+SH
+Text Label 1500 4650 2    50   ~ 0
+SU
 Text Label 1500 5850 2    50   ~ 0
-SX
+SI
+Text Label 4050 5400 0    50   ~ 0
+SO
+Text Label 1500 6150 2    50   ~ 0
+SJ
+Text Label 4050 4500 0    50   ~ 0
+SL
+Text Label 1500 5400 2    50   ~ 0
+SN
+Text Label 4050 4950 0    50   ~ 0
+SK
 Text Label 4050 5700 0    50   ~ 0
-SD
-Text Label 4050 6000 0    50   ~ 0
-SR
+SE
+Text Label 1500 6000 2    50   ~ 0
+SA
 Text Label 4050 5250 0    50   ~ 0
-SC
-Text Label 1500 4650 2    50   ~ 0
-SV
-Text Label 1500 6000 2    50   ~ 0
-SB
+SS
+Text Label 1500 5100 2    50   ~ 0
+SP
+Text Label 1500 5700 2    50   ~ 0
+ST
 Text Label 4050 5550 0    50   ~ 0
-SH
-Text Label 4050 5850 0    50   ~ 0
-SU
-Text Label 4050 4650 0    50   ~ 0
-SI
-Text Label 1500 5250 2    50   ~ 0
-SO
-Text Label 3450 4200 1    50   ~ 0
-SJ
-Text Label 1500 6150 2    50   ~ 0
-SL
-Text Label 4050 5100 0    50   ~ 0
-SN
-Text Label 1500 5700 2    50   ~ 0
-SK
-Text Label 1500 4950 2    50   ~ 0
-SE
-Text Label 4050 4500 0    50   ~ 0
-SA
-Text Label 1500 5400 2    50   ~ 0
-SS
-Text Label 4050 5400 0    50   ~ 0
-SP
-Text Label 4050 4800 0    50   ~ 0
-ST
-Text Label 1500 5100 2    50   ~ 0
 SZ
 Text Label 3600 4200 1    50   ~ 0
 SF
-Text Label 1500 5550 2    50   ~ 0
+Text Label 4050 5100 0    50   ~ 0
 SG
-Text Label 1500 4800 2    50   ~ 0
+Text Label 4050 5850 0    50   ~ 0
 SM
 Text Label 6550 5100 3    50   ~ 0
@@
 Text Label 5200 5100 3    50   ~ 0
 SP
-Text Label 4050 6150 0    50   ~ 0
+Text Label 1950 4200 1    50   ~ 0
 SQ
-Text Label 4050 4950 0    50   ~ 0
+Text Label 1500 5550 2    50   ~ 0
 SW
 NoConn ~ 3000 4200
@@
 	1    0    0    -1
 $EndComp
-NoConn ~ 1950 4200
-NoConn ~ 2100 4200
 NoConn ~ 2250 4200
 NoConn ~ 2400 4200
@@
 Text Label 10000 3275 0    50   ~ 0
 SB
+NoConn ~ 3450 4200
+NoConn ~ 2100 4200
 $EndSCHEMATC
