File: PCB/plugboard.kicad_pcb (KiCad board)
At the start: 2 copper layers, 94 parts, among them J1 1/4" Jack, J10 Conn_01x19_Male_0, J11 Conn_01x19_Male_0, J2 1/4" Jack, J3 1/4" Jack, J4 1/4" Jack, J5 1/4" Jack, J6 1/4" Jack, J7 1/4" Jack, J8 1/4" Jack, J9 1/4" Jack, P1 CONN_02X03, P2 CONN_02X03

Commit message: Basic Layout
Now I'm gonna start on tracing.
Parts:
- added R81: R_10K, enigmaprints:R_0805_OEM, F.Cu at (118.7, 68.7)
- added U1: ADG732, enigmaprints:ADG732BSUZ-REEL, F.Cu at (156.1, 88.8)
- J10: value Conn_01x19_Male_0 -> 1/4" Jack; footprint enigmaprints:sidebar -> enigmaprints:jack_hole
- J7: value 1/4" Jack -> Conn_01x19_Male_0; footprint enigmaprints:jack_hole -> enigmaprints:sidebar
- R11, R9: value R_10K -> R_1K
- R15, R16, R17, R18, R19, R20, R21, R22, R23, R24, R26: value R_0 -> R_1K
- R32, R33, R40, R53, R54, R61, R68, R75, R76, R77, R78, R79: value R_1K -> R_0
- R45: value R_0 -> R_10K
- R80: value R_1K -> R_10K
- moved J10 157.4 mm to (167.9, 156.2)
- moved R25 142.1 mm to (170.5, 176.0), turned to 90 degrees
- moved R26 141.6 mm to (173.2, 176.0), turned to 270 degrees
- moved R23 141.0 mm to (165.1, 176.0), turned to 90 degrees
- moved R22 139.5 mm to (162.4, 176.0), turned to 270 degrees
- moved R24 139.4 mm to (167.8, 176.0), turned to 270 degrees
- moved R18 137.8 mm to (151.5, 176.0), turned to 270 degrees
- moved R19 137.4 mm to (154.2, 176.0), turned to 90 degrees
- moved R21 136.5 mm to (159.7, 176.0), turned to 90 degrees
- moved R20 133.6 mm to (157.0, 176.0), turned to 270 degrees
- moved R17 131.0 mm to (148.8, 176.0), turned to 90 degrees
- moved R15 130.1 mm to (143.4, 176.0), turned to 90 degrees
- moved R16 129.9 mm to (146.1, 176.0), turned to 270 degrees
- moved R13 129.4 mm to (138.0, 176.0), turned to 90 degrees
- moved R14 129.2 mm to (140.7, 176.0), turned to 270 degrees
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Connections:
- J10 pad 1: /S1 -> Net-(J10-Pad1)
- J10 pad 2: /S6 -> Net-(J10-Pad2)
- J10 pad 3: /S2 -> Net-(J10-Pad3)
- J10 pad 4: /S4 -> (no net)
- J10 pad 5: /S7 -> (no net)
- J11 pad 1: /S1 -> /SQ
- J11 pad 10: /S9 -> /SD
- J11 pad 11: /S15 -> /SC
- J11 pad 12: /S11 -> /ST
- J11 pad 13: /S13 -> /SF
- J11 pad 14: /S16 -> /SV
- J11 pad 15: /S12 -> /SZ
- J11 pad 16: /S14 -> /SG
- J11 pad 17: /S17 -> /SB
- J11 pad 2: /S6 -> /SP
- J11 pad 3: /S2 -> /SW
- J11 pad 4: /S4 -> /SA
- J11 pad 5: /S7 -> /SY
- J11 pad 6: /S3 -> /SE
- J11 pad 7: /S5 -> /SS
- J11 pad 8: /S8 -> /SX
- J11 pad 9: /S10 -> /SR
- J7 pad 1: Net-(J7-Pad1) -> /SQ
- J7 pad 2: Net-(J7-Pad2) -> /SP
- J7 pad 3: Net-(J7-Pad3) -> /SW
- J7 pad 4: (no net) -> /SA
- J7 pad 5: (no net) -> /SY
- R10 pad 1: /J -> /K
- R10 pad 2: /I -> /J
- R11 pad 1: VCC -> /L
- R11 pad 2: /~CS -> /K
- R12 pad 1: /K -> /M
- R12 pad 2: /J -> /L
- R13 pad 1: /L -> /N
- R13 pad 2: /K -> /M
- R14 pad 1: /M -> /O
- R14 pad 2: /L -> /N
- R15 pad 1: Net-(J1-Pad1) -> /P
- R15 pad 2: /Q -> /O
- R16 pad 1: Net-(J1-Pad3) -> /Q
- R16 pad 2: /S1 -> /P
- R17 pad 1: /P -> /R
- R17 pad 2: Net-(J3-Pad1) -> /Q
- R18 pad 1: Net-(J3-Pad3) -> /S
- R18 pad 2: /S6 -> /R
- R19 pad 1: Net-(J1-Pad1) -> /T
- R19 pad 2: /R -> /S
- R20 pad 1: Net-(J1-Pad3) -> /U
- R20 pad 2: /S10 -> /T
- R21 pad 1: /D -> /V
- R21 pad 2: Net-(J2-Pad1) -> /U
- R22 pad 1: Net-(J2-Pad3) -> /W
- R22 pad 2: /S9 -> /V
- R23 pad 1: /C -> /X
- R23 pad 2: Net-(J3-Pad1) -> /W
- R24 pad 1: Net-(J3-Pad3) -> /Y
- R24 pad 2: /S15 -> /X
- R25 pad 1: /N -> /Z
- R25 pad 2: /M -> /Y
- R26 pad 1: Net-(J1-Pad1) -> GND
- R26 pad 2: /U -> /Z
- R27 pad 1: Net-(J1-Pad3) -> Net-(J1-Pad1)
- R27 pad 2: /S19 -> /Q
- R28 pad 1: /H -> Net-(J1-Pad1)
- R28 pad 2: Net-(J2-Pad1) -> /R
- R29 pad 1: Net-(J2-Pad3) -> Net-(J1-Pad1)
- R29 pad 2: /S18 -> /U
- R30 pad 1: /N -> Net-(J2-Pad1)
- R30 pad 2: Net-(J3-Pad1) -> /W
- R31 pad 1: Net-(J3-Pad3) -> Net-(J2-Pad1)
- R31 pad 2: /S24 -> /T
- R32 pad 1: /O -> Net-(J2-Pad1)
- R32 pad 2: /N -> /I
- R33 pad 1: /P -> Net-(J3-Pad1)
- R33 pad 2: /O -> /E
- R34 pad 1: Net-(J4-Pad1) -> Net-(J3-Pad1)
- R34 pad 2: /W -> /Z
- R35 pad 1: Net-(J4-Pad3) -> Net-(J3-Pad1)
- R35 pad 2: /S2 -> /O
- R36 pad 1: VCC -> Net-(J1-Pad3)
- R36 pad 2: Net-(J5-Pad1) -> /SQ
- R37 pad 1: Net-(J5-Pad3) -> Net-(J1-Pad3)
- R37 pad 2: /S4 -> /SR
- R38 pad 1: /Y -> Net-(J1-Pad3)
- R38 pad 2: Net-(J6-Pad1) -> /SU
- R39 pad 1: Net-(J6-Pad3) -> Net-(J2-Pad3)
- R39 pad 2: /S7 -> /SW
- R40 pad 1: /Q -> Net-(J2-Pad3)
- R40 pad 2: /P -> /ST
- R41 pad 1: Net-(J4-Pad1) -> Net-(J2-Pad3)
- R41 pad 2: /T -> /SI
- R42 pad 1: Net-(J4-Pad3) -> Net-(J3-Pad3)
- R42 pad 2: /S11 -> /SE
- R43 pad 1: /F -> Net-(J3-Pad3)
- R43 pad 2: Net-(J5-Pad1) -> /SZ
- R44 pad 1: Net-(J5-Pad3) -> Net-(J3-Pad3)
- R44 pad 2: /S13 -> /SO
- R45 pad 1: /V -> /Dout
- R45 pad 2: Net-(J6-Pad1) -> GND
- R46 pad 1: Net-(J6-Pad3) -> /D
- R46 pad 2: /S16 -> Net-(J4-Pad1)
- R47 pad 1: Net-(J4-Pad1) -> /H
- R47 pad 2: /I -> Net-(J4-Pad1)
- R48 pad 1: Net-(J4-Pad3) -> VCC
- R48 pad 2: /S20 -> Net-(J5-Pad1)
- R49 pad 1: /J -> /F
- R50 pad 1: Net-(J5-Pad3) -> /J
- R50 pad 2: /S22 -> Net-(J5-Pad1)
- R51 pad 1: /M -> /S
- R52 pad 1: Net-(J6-Pad3) -> /G
- R52 pad 2: /S25 -> Net-(J6-Pad1)
- R53 pad 1: /R -> /K
- R53 pad 2: /Q -> Net-(J6-Pad1)
- R54 pad 1: /S -> Net-(J4-Pad3)
- R54 pad 2: /R -> /SD
- R55 pad 1: Net-(J7-Pad1) -> Net-(J4-Pad3)
- R55 pad 2: /E -> /SH
- R56 pad 1: Net-(J7-Pad3) -> Net-(J5-Pad3)
- R56 pad 2: /S3 -> /SA
- R57 pad 1: /S -> Net-(J5-Pad3)
- R57 pad 2: Net-(J8-Pad1) -> /SF
- R58 pad 1: Net-(J8-Pad3) -> Net-(J5-Pad3)
- R58 pad 2: /S5 -> /SJ
- R59 pad 1: /X -> Net-(J6-Pad3)
- R59 pad 2: Net-(J9-Pad1) -> /SS
- R60 pad 1: Net-(J9-Pad3) -> Net-(J6-Pad3)
- R60 pad 2: /S8 -> /SG
- R61 pad 1: /T -> Net-(J6-Pad3)
- R61 pad 2: /S -> /SK
- R62 pad 1: Net-(J7-Pad1) -> /P
- R62 pad 2: /Z -> Net-(J8-Pad1)
- R63 pad 1: Net-(J7-Pad3) -> /C
- R63 pad 2: /S12 -> Net-(J8-Pad1)
- R64 pad 1: /G -> /N
- R65 pad 1: Net-(J8-Pad3) -> /Y
- R65 pad 2: /S14 -> Net-(J9-Pad1)
- R66 pad 1: /B -> /V
- R67 pad 1: Net-(J9-Pad3) -> /M
- R67 pad 2: /S17 -> Net-(J9-Pad1)
- R68 pad 1: /U -> /X
- R68 pad 2: /T -> Net-(J10-Pad1)
- R69 pad 1: Net-(J7-Pad1) -> /B
- R69 pad 2: /O -> Net-(J10-Pad1)
- R70 pad 1: Net-(J7-Pad3) -> /L
- R70 pad 2: /S21 -> Net-(J10-Pad1)
- R71 pad 1: /K -> Net-(J8-Pad3)
- R71 pad 2: Net-(J8-Pad1) -> /SP
- R72 pad 2: /S23 -> /SC
- R73 pad 1: /L -> Net-(J8-Pad3)
- R73 pad 2: Net-(J9-Pad1) -> /SN
- R74 pad 2: /S26 -> /SY
- R75 pad 1: /V -> Net-(J9-Pad3)
- R75 pad 2: /U -> /SV
- R76 pad 1: /W -> Net-(J9-Pad3)
- R76 pad 2: /V -> /SM
- R77 pad 1: /X -> Net-(J10-Pad3)
- R77 pad 2: /W -> /SX
- R78 pad 1: /Y -> Net-(J10-Pad3)
- R78 pad 2: /X -> /SB
- R79 pad 1: /Z -> Net-(J10-Pad3)
- R79 pad 2: /Y -> /SL
- R80 pad 1: GND -> VCC
- R80 pad 2: /Z -> /~EN
- R9 pad 1: VCC -> /J
- R9 pad 2: /~EN -> /I
Other:
- board outline added: 100 x 100 mm

Commit message: update schematic
I'm gonna try something...
Parts:
- moved U1 16.4 mm to (139.7, 88.4), turned to 180 degrees
- moved R46 0.89 mm to (122.4, 124.8), turned to 180 degrees
- moved R47 0.89 mm to (122.4, 127.1), turned to 180 degrees
- moved R62 0.76 mm to (122.4, 148.1), turned to 180 degrees
- moved R63 0.76 mm to (122.4, 150.5), turned to 180 degrees
- moved R64 0.76 mm to (122.4, 152.8), turned to 180 degrees
- moved R54 0.64 mm to (122.4, 131.9)
- moved R55 0.64 mm to (122.4, 134.2)
- moved R71 0.63 mm to (122.4, 156.4)
- moved R72 0.63 mm to (122.4, 158.7)
- moved R73 0.63 mm to (122.4, 161.1)
- moved R27 0.25 mm to (122.4, 98.7)
- moved R28 0.25 mm to (122.4, 101.0)
- moved R29 0.25 mm to (122.4, 103.3)
- moved R36 0.13 mm to (122.4, 106.7)
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Connections:
- R1 pad 1: /B -> /R
- R10 pad 1: /K -> /I
- R10 pad 2: /J -> /T
- R11 pad 1: /L -> /A
- R11 pad 2: /K -> /I
- R12 pad 1: /M -> /F
- R12 pad 2: /L -> /A
- R13 pad 1: /N -> /J
- R13 pad 2: /M -> /F
- R14 pad 1: /O -> /Y
- R14 pad 2: /N -> /J
- R15 pad 1: /P -> /V
- R15 pad 2: /O -> /Y
- R16 pad 1: /Q -> /M
- R16 pad 2: /P -> /V
- R17 pad 1: /R -> /E
- R17 pad 2: /Q -> /M
- R18 pad 1: /S -> /Z
- R18 pad 2: /R -> /E
- R19 pad 1: /T -> /O
- R19 pad 2: /S -> /Z
- R2 pad 1: /C -> /U
- R2 pad 2: /B -> /R
- R20 pad 1: /U -> /S
- R20 pad 2: /T -> /O
- R21 pad 1: /V -> /G
- R21 pad 2: /U -> /S
- R22 pad 1: /W -> /K
- R22 pad 2: /V -> /G
- R23 pad 2: /W -> /K
- R24 pad 1: /Y -> /B
- R25 pad 1: /Z -> /L
- R25 pad 2: /Y -> /B
- R26 pad 2: /Z -> /L
- R27 pad 2: /Q -> VCC
- R3 pad 2: /C -> /U
- R4 pad 1: /E -> /H
- R48 pad 1: VCC -> /A
- R5 pad 1: /F -> /P
- R5 pad 2: /E -> /H
- R6 pad 1: /G -> /C
- R6 pad 2: /F -> /P
- R7 pad 1: /H -> /N
- R7 pad 2: /G -> /C
- R8 pad 1: /I -> /W
- R8 pad 2: /H -> /N
- R9 pad 1: /J -> /T
- R9 pad 2: /I -> /W
- U1 pad 1: /SZ -> /SS
- U1 pad 10: /SE -> Net-(U1-Pad10)
- U1 pad 11: /SW -> Net-(U1-Pad11)
- U1 pad 12: /SQ -> Net-(U1-Pad12)
- U1 pad 2: /ST -> /SG
- U1 pad 25: /SB -> /SQ
- U1 pad 26: /SH -> /SR
- U1 pad 28: /SI -> /SD
- U1 pad 29: /SO -> /SH
- U1 pad 3: /SR -> /SK
- U1 pad 30: /SJ -> /SP
- U1 pad 31: /SK -> /SC
- U1 pad 33: /SM -> /SW
- U1 pad 34: /SL -> /ST
- U1 pad 35: Net-(U1-Pad35) -> /SI
- U1 pad 36: Net-(U1-Pad36) -> /SA
- U1 pad 37: Net-(U1-Pad37) -> /SF
- U1 pad 38: Net-(U1-Pad38) -> /SJ
- U1 pad 39: Net-(U1-Pad39) -> /SY
- U1 pad 4: /SD -> /SX
- U1 pad 40: Net-(U1-Pad40) -> /SV
- U1 pad 45: /SV -> /SM
- U1 pad 46: /SC -> /SE
- U1 pad 47: /SG -> /SZ
- U1 pad 48: /SF -> /SO
- U1 pad 5: /SX -> /SB
- U1 pad 6: /SY -> /SL
- U1 pad 7: /SP -> Net-(U1-Pad7)
- U1 pad 8: /SS -> Net-(U1-Pad8)
- U1 pad 9: /SA -> Net-(U1-Pad9)
Routing:
- net /SP: track 0.00 -> 115.3 mm, vias 0 -> 2
- net /SC: track 0.00 -> 80.3 mm
- net /SN: track 0.00 -> 80.1 mm
- net /SQ: track 0.00 -> 64.8 mm
- net /SH: track 0.00 -> 56.9 mm
- net /SD: track 0.00 -> 55.0 mm
- net /SI: track 0.00 -> 41.6 mm
- net /ST: track 0.00 -> 40.4 mm
- net /SW: track 0.00 -> 39.8 mm
- net /SU: track 0.00 -> 35.3 mm
- net /SR: track 0.00 -> 33.0 mm
- net Net-(J1-Pad1): track 0.00 -> 23.8 mm
- net Net-(J8-Pad1): track 0.00 -> 22.2 mm
- net Net-(J2-Pad1): track 0.00 -> 20.5 mm
- net Net-(J4-Pad1): track 0.00 -> 20.2 mm
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Other:
- net class Default: clearance 0.2 -> 0.1524; trace_width 0.25 -> 0.1524; via_dia 0.8 -> 0.6096; via_drill 0.4 -> 0.3048
- rule trace_clearance: 0.2 -> 0.1524
- rule trace_min: 0.2 -> 0.1524
- rule via_min_drill: 0.3 -> 0.3048
- rule via_min_size: 0.4 -> 0.6096

Commit message: More Layout
I think it's working...
Parts:
- moved R33 76.5 mm to (151.6, 169.2), turned to 270 degrees
- moved R30 74.8 mm to (127.1, 169.2), turned to 270 degrees
- moved R34 73.4 mm to (154.3, 169.2), turned to 270 degrees
- moved R27 72.5 mm to (105.3, 169.2), turned to 270 degrees
- moved R31 71.7 mm to (129.8, 169.2), turned to 270 degrees
- moved R35 70.3 mm to (157.0, 169.2), turned to 270 degrees
- moved R28 69.7 mm to (108.0, 169.2), turned to 270 degrees
- moved R32 68.7 mm to (132.5, 169.2), turned to 270 degrees
- moved R29 66.8 mm to (110.7, 169.2), turned to 270 degrees
- moved R51 50.6 mm to (159.7, 169.2), turned to 90 degrees
- moved R48 48.1 mm to (135.2, 169.2), turned to 90 degrees
- moved R52 47.5 mm to (162.5, 169.2), turned to 90 degrees
- moved R46 45.3 mm to (113.5, 169.2), turned to 90 degrees
- moved R49 45.1 mm to (138.0, 169.2), turned to 90 degrees
- moved R53 44.3 mm to (165.2, 169.2), turned to 90 degrees
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Routing:
- net /SP: track 115.3 -> 0.00 mm, vias 2 -> 0
- net /SC: track 80.3 -> 0.00 mm
- net /SN: track 80.1 -> 0.00 mm
- net Net-(J3-Pad1): track 0.00 -> 73.5 mm
- net /SQ: track 64.8 -> 0.00 mm
- net /SH: track 56.9 -> 0.00 mm
- net /SD: track 55.0 -> 0.00 mm
- net Net-(J2-Pad1): track 20.5 -> 74.0 mm
- net Net-(J1-Pad1): track 23.8 -> 75.6 mm
- net Net-(J5-Pad1): track 0.00 -> 50.6 mm
- net Net-(J6-Pad1): track 0.00 -> 49.4 mm
- net /SI: track 41.6 -> 0.00 mm
- net /ST: track 40.4 -> 0.00 mm
- net /SW: track 39.8 -> 0.00 mm
- net /SU: track 35.3 -> 0.00 mm
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