File: wire_power/wire_power.sch (KiCad schematic (older format))
At the start: 34 parts

Commit message: Updates letter labelling relays
Parts:
- C?: symbol formula:C_0.1uF -> wire_power-rescue:C_0.1uF-formula
- J? (x3): symbol formula:CONN_02X03 -> wire_power-rescue:CONN_02X03-formula
- Q? (x26): symbol Enigma:CPC1025NTR -> wire_power-rescue:CPC1025NTR-Enigma
- R? (x2): symbol formula:R_10K -> wire_power-rescue:R_10K-formula
- R?: symbol formula:R_200 -> wire_power-rescue:R_200-formula
- U?: symbol Enigma:ADG732 -> wire_power-rescue:ADG732-Enigma
Connections:
- net labels added: Hot_outA, Hot_outB, Hot_outC, Hot_outD, Hot_outE, Hot_outF, Hot_outG, Hot_outH, Hot_outI, Hot_outJ, Hot_outK, Hot_outL, Hot_outM, Hot_outN, Hot_outO, Hot_outP, Hot_outQ, Hot_outR, Hot_outS, Hot_outT, Hot_outU, Hot_outV, Hot_outW, Hot_outX, Hot_outY, Hot_outZ
Changed lines of the file:
@@
 $EndDescr
 $Comp
-L formula:CONN_02X03 J?
+L wire_power-rescue:CONN_02X03-formula J?
 U 1 1 5BEB666D
 P 1500 1300
@@
 $EndComp
 $Comp
-L formula:CONN_02X03 J?
+L wire_power-rescue:CONN_02X03-formula J?
 U 1 1 5BEB6B2A
 P 1500 1900
@@
 $EndComp
 $Comp
-L Enigma:ADG732 U?
+L wire_power-rescue:ADG732-Enigma U?
 U 1 1 5BEB6C8D
 P 2750 6150
@@
 $EndComp
 $Comp
-L Enigma:CPC1025NTR Q?
+L wire_power-rescue:CPC1025NTR-Enigma Q?
 U 1 1 5BEB70D3
 P 5700 1400
@@
 $EndComp
 $Comp
-L formula:R_10K R?
+L wire_power-rescue:R_10K-formula R?
 U 1 1 5BEBE0C3
 P 4150 6800
@@
 $EndComp
 $Comp
-L formula:R_10K R?
+L wire_power-rescue:R_10K-formula R?
 U 1 1 5BEBE170
 P 4550 6800
@@
 ~EN
 $Comp
-L formula:C_0.1uF C?
+L wire_power-rescue:C_0.1uF-formula C?
 U 1 1 5BEC5B93
 P 2250 6850
@@
 $EndComp
 $Comp
-L formula:R_200 R?
+L wire_power-rescue:R_200-formula R?
 U 1 1 5BEC7F2C
 P 3000 3950
@@
 	3000 4100 3000 4250
 $Comp
-L formula:CONN_02X03 J?
+L wire_power-rescue:CONN_02X03-formula J?
 U 1 1 5BEC8EA9
 P 1500 2550
@@
 Hot_in
 Text Label 6000 1500 0    50   ~ 0
-Hot_out
+Hot_outA
 Wire Wire Line
 	5400 1500 5300 1500
@@
 SZ
 $Comp
-L Enigma:CPC1025NTR Q?
+L wire_power-rescue:CPC1025NTR-Enigma Q?
 U 1 1 5BED7AAE
 P 6800 1400
@@
 Hot_in
 Text Label 7100 1500 0    50   ~ 0
-Hot_out
+Hot_outB
 Wire Wire Line
 	6500 1500 6400 1500
@@
 	6400 1500 6400 1550
 $Comp
-L Enigma:CPC1025NTR Q?
+L wire_power-rescue:CPC1025NTR-Enigma Q?
 U 1 1 5BED86EE
 P 7900 1400
@@
 Hot_in
 Text Label 8200 1500 0    50   ~ 0
-Hot_out
+Hot_outC
 Wire Wire Line
 	7600 1500 7500 1500
@@
 	7500 1500 7500 1550
 $Comp
-L Enigma:CPC1025NTR Q?
+L wire_power-rescue:CPC1025NTR-Enigma Q?
 U 1 1 5BED86FF
 P 9000 1400
@@
 Hot_in
 Text Label 9300 1500 0    50   ~ 0
-Hot_out
+Hot_outD
 Wire Wire Line
 	8700 1500 8600 1500
@@
 	8600 1500 8600 1550
 $Comp
-L Enigma:CPC1025NTR Q?
+L wire_power-rescue:CPC1025NTR-Enigma Q?
 U 1 1 5BED8D94
 P 5700 2000
@@
 Hot_in
 Text Label 6000 2100 0    50   ~ 0
-Hot_out
+Hot_outE
 Wire Wire Line
 	5400 2100 5300 2100
@@
 	5300 2100 5300 2150
 $Comp
-L Enigma:CPC1025NTR Q?
+L wire_power-rescue:CPC1025NTR-Enigma Q?
 U 1 1 5BED8DA5
 P 6800 2000
@@
 Hot_in
 Text Label 7100 2100 0    50   ~ 0
-Hot_out
+Hot_outF
 Wire Wire Line
 	6500 2100 6400 2100
@@
 	6400 2100 6400 2150
 $Comp
-L Enigma:CPC1025NTR Q?
+L wire_power-rescue:CPC1025NTR-Enigma Q?
 U 1 1 5BED8DB6
 P 7900 2000
@@
 Hot_in
 Text Label 8200 2100 0    50   ~ 0
-Hot_out
+Hot_outG
 Wire Wire Line
 	7600 2100 7500 2100
@@
 	7500 2100 7500 2150
 $Comp
-L Enigma:CPC1025NTR Q?
+L wire_power-rescue:CPC1025NTR-Enigma Q?
 U 1 1 5BED8DC7
 P 9000 2000
@@
 Hot_in
 Text Label 9300 2100 0    50   ~ 0
-Hot_out
+Hot_outH
 Wire Wire Line
 	8700 2100 8600 2100
@@
 	8600 2100 8600 2150
 $Comp
-L Enigma:CPC1025NTR Q?
+L wire_power-rescue:CPC1025NTR-Enigma Q?
 U 1 1 5BED987C
 P 5700 2600
@@
 Hot_in
 Text Label 6000 2700 0    50   ~ 0
-Hot_out
+Hot_outI
 Wire Wire Line
 	5400 2700 5300 2700
@@
 	5300 2700 5300 2750
 $Comp
-L Enigma:CPC1025NTR Q?
+L wire_power-rescue:CPC1025NTR-Enigma Q?
 U 1 1 5BED988D
 P 6800 2600
@@
 Hot_in
 Text Label 7100 2700 0    50   ~ 0
-Hot_out
+Hot_outJ
 Wire Wire Line
 	6500 2700 6400 2700
@@
 	6400 2700 6400 2750
 $Comp
-L Enigma:CPC1025NTR Q?
+L wire_power-rescue:CPC1025NTR-Enigma Q?
 U 1 1 5BED989E
 P 7900 2600
@@
 Hot_in
 Text Label 8200 2700 0    50   ~ 0
-Hot_out
+Hot_outK
 Wire Wire Line
 	7600 2700 7500 2700
@@
 	7500 2700 7500 2750
 $Comp
-L Enigma:CPC1025NTR Q?
+L wire_power-rescue:CPC1025NTR-Enigma Q?
 U 1 1 5BED98AF
 P 9000 2600
@@
 Hot_in
 Text Label 9300 2700 0    50   ~ 0
-Hot_out
+Hot_outL
 Wire Wire Line
 	8700 2700 8600 2700
@@
 	8600 2700 8600 2750
 $Comp
-L Enigma:CPC1025NTR Q?
+L wire_power-rescue:CPC1025NTR-Enigma Q?
 U 1 1 5BED98C0
 P 5700 3200
@@
 Hot_in
 Text Label 6000 3300 0    50   ~ 0
-Hot_out
+Hot_outM
 Wire Wire Line
 	5400 3300 5300 3300
@@
 	5300 3300 5300 3350
 $Comp
-L Enigma:CPC1025NTR Q?
+L wire_power-rescue:CPC1025NTR-Enigma Q?
 U 1 1 5BED98D1
 P 6800 3200
@@
 Hot_in
 Text Label 7100 3300 0    50   ~ 0
-Hot_out
+Hot_outN
 Wire Wire Line
 	6500 3300 6400 3300
@@
 	6400 3300 6400 3350
 $Comp
-L Enigma:CPC1025NTR Q?
+L wire_power-rescue:CPC1025NTR-Enigma Q?
 U 1 1 5BED98E2
 P 7900 3200
@@
 Hot_in
 Text Label 8200 3300 0    50   ~ 0
-Hot_out
+Hot_outO
 Wire Wire Line
 	7600 3300 7500 3300
@@
 	7500 3300 7500 3350
 $Comp
-L Enigma:CPC1025NTR Q?
+L wire_power-rescue:CPC1025NTR-Enigma Q?
 U 1 1 5BED98F3
 P 9000 3200
@@
 Hot_in
 Text Label 9300 3300 0    50   ~ 0
-Hot_out
+Hot_outP
 Wire Wire Line
 	8700 3300 8600 3300
@@
 	8600 3300 8600 3350
 $Comp
-L Enigma:CPC1025NTR Q?
+L wire_power-rescue:CPC1025NTR-Enigma Q?
 U 1 1 5BEDAE9E
 P 5700 3850
@@
 Hot_in
 Text Label 6000 3950 0    50   ~ 0
-Hot_out
+Hot_outQ
 Wire Wire Line
 	5400 3950 5300 3950
@@
 	5300 3950 5300 4000
 $Comp
-L Enigma:CPC1025NTR Q?
+L wire_power-rescue:CPC1025NTR-Enigma Q?
 U 1 1 5BEDAEAF
 P 6800 3850
@@
 Hot_in
 Text Label 7100 3950 0    50   ~ 0
-Hot_out
+Hot_outR
 Wire Wire Line
 	6500 3950 6400 3950
@@
 	6400 3950 6400 4000
 $Comp
-L Enigma:CPC1025NTR Q?
+L wire_power-rescue:CPC1025NTR-Enigma Q?
 U 1 1 5BEDAEC0
 P 7900 3850
@@
 Hot_in
 Text Label 8200 3950 0    50   ~ 0
-Hot_out
+Hot_outS
 Wire Wire Line
 	7600 3950 7500 3950
@@
 	7500 3950 7500 4000
 $Comp
-L Enigma:CPC1025NTR Q?
+L wire_power-rescue:CPC1025NTR-Enigma Q?
 U 1 1 5BEDAED1
 P 9000 3850
@@
 Hot_in
 Text Label 9300 3950 0    50   ~ 0
-Hot_out
+Hot_outT
 Wire Wire Line
 	8700 3950 8600 3950
@@
 	8600 3950 8600 4000
 $Comp
-L Enigma:CPC1025NTR Q?
+L wire_power-rescue:CPC1025NTR-Enigma Q?
 U 1 1 5BEDAEE2
 P 5700 4450
@@
 Hot_in
 Text Label 6000 4550 0    50   ~ 0
-Hot_out
+Hot_outU
 Wire Wire Line
 	5400 4550 5300 4550
@@
 	5300 4550 5300 4600
 $Comp
-L Enigma:CPC1025NTR Q?
+L wire_power-rescue:CPC1025NTR-Enigma Q?
 U 1 1 5BEDAEF3
 P 6800 4450
@@
 Hot_in
 Text Label 7100 4550 0    50   ~ 0
-Hot_out
+Hot_outV
 Wire Wire Line
 	6500 4550 6400 4550
@@
 	6400 4550 6400 4600
 $Comp
-L Enigma:CPC1025NTR Q?
+L wire_power-rescue:CPC1025NTR-Enigma Q?
 U 1 1 5BEDAF04
 P 7900 4450
@@
 Hot_in
 Text Label 8200 4550 0    50   ~ 0
-Hot_out
+Hot_outW
 Wire Wire Line
 	7600 4550 7500 4550
@@
 	7500 4550 7500 4600
 $Comp
-L Enigma:CPC1025NTR Q?
+L wire_power-rescue:CPC1025NTR-Enigma Q?
 U 1 1 5BEDAF15
 P 9000 4450
@@
 Hot_in
 Text Label 9300 4550 0    50   ~ 0
-Hot_out
+Hot_outX
 Wire Wire Line
 	8700 4550 8600 4550
@@
 	8600 4550 8600 4600
 $Comp
-L Enigma:CPC1025NTR Q?
+L wire_power-rescue:CPC1025NTR-Enigma Q?
 U 1 1 5BEDF896
 P 6800 5050
@@
 Hot_in
 Text Label 7100 5150 0    50   ~ 0
-Hot_out
+Hot_outY
 Wire Wire Line
 	6500 5150 6400 5150
@@
 	6400 5150 6400 5200
 $Comp
-L Enigma:CPC1025NTR Q?
+L wire_power-rescue:CPC1025NTR-Enigma Q?
 U 1 1 5BEDF8A7
 P 7900 5050
@@
 Hot_in
 Text Label 8200 5150 0    50   ~ 0
-Hot_out
+Hot_outZ
 Wire Wire Line
 	7600 5150 7500 5150

Commit message: Fix schematic
Parts:
- added J?: Conn_01x26_Male_0, symbol enigma:Conn_01x26_Male_0
- C?: symbol wire_power-rescue:C_0.1uF-formula -> formula:C_0.1uF
- J? (x3): symbol wire_power-rescue:CONN_02X03-formula -> formula:CONN_02X03
- Q? (x26): symbol wire_power-rescue:CPC1025NTR-Enigma -> enigma:CPC1025NTR
- R? (x2): symbol wire_power-rescue:R_10K-formula -> formula:R_10K
- R?: symbol wire_power-rescue:R_200-formula -> formula:R_200
- U?: symbol wire_power-rescue:ADG732-Enigma -> enigma:ADG732
Changed lines of the file:
@@
 $EndDescr
 $Comp
-L wire_power-rescue:CONN_02X03-formula J?
+L formula:CONN_02X03 J?
 U 1 1 5BEB666D
 P 1500 1300
@@
 $EndComp
 $Comp
-L wire_power-rescue:CONN_02X03-formula J?
+L formula:CONN_02X03 J?
 U 1 1 5BEB6B2A
 P 1500 1900
@@
 $EndComp
 $Comp
-L wire_power-rescue:ADG732-Enigma U?
+L enigma:ADG732 U?
 U 1 1 5BEB6C8D
 P 2750 6150
@@
 $EndComp
 $Comp
-L wire_power-rescue:CPC1025NTR-Enigma Q?
+L enigma:CPC1025NTR Q?
 U 1 1 5BEB70D3
 P 5700 1400
@@
 $EndComp
 $Comp
-L wire_power-rescue:R_10K-formula R?
+L formula:R_10K R?
 U 1 1 5BEBE0C3
 P 4150 6800
@@
 $EndComp
 $Comp
-L wire_power-rescue:R_10K-formula R?
+L formula:R_10K R?
 U 1 1 5BEBE170
 P 4550 6800
@@
 ~EN
 $Comp
-L wire_power-rescue:C_0.1uF-formula C?
+L formula:C_0.1uF C?
 U 1 1 5BEC5B93
 P 2250 6850
@@
 $EndComp
 $Comp
-L wire_power-rescue:R_200-formula R?
+L formula:R_200 R?
 U 1 1 5BEC7F2C
 P 3000 3950
@@
 	3000 4100 3000 4250
 $Comp
-L wire_power-rescue:CONN_02X03-formula J?
+L formula:CONN_02X03 J?
 U 1 1 5BEC8EA9
 P 1500 2550
@@
 SZ
 $Comp
-L wire_power-rescue:CPC1025NTR-Enigma Q?
+L enigma:CPC1025NTR Q?
 U 1 1 5BED7AAE
 P 6800 1400
@@
 	6400 1500 6400 1550
 $Comp
-L wire_power-rescue:CPC1025NTR-Enigma Q?
+L enigma:CPC1025NTR Q?
 U 1 1 5BED86EE
 P 7900 1400
@@
 	7500 1500 7500 1550
 $Comp
-L wire_power-rescue:CPC1025NTR-Enigma Q?
+L enigma:CPC1025NTR Q?
 U 1 1 5BED86FF
 P 9000 1400
@@
 	8600 1500 8600 1550
 $Comp
-L wire_power-rescue:CPC1025NTR-Enigma Q?
+L enigma:CPC1025NTR Q?
 U 1 1 5BED8D94
 P 5700 2000
@@
 	5300 2100 5300 2150
 $Comp
-L wire_power-rescue:CPC1025NTR-Enigma Q?
+L enigma:CPC1025NTR Q?
 U 1 1 5BED8DA5
 P 6800 2000
@@
 	6400 2100 6400 2150
 $Comp
-L wire_power-rescue:CPC1025NTR-Enigma Q?
+L enigma:CPC1025NTR Q?
 U 1 1 5BED8DB6
 P 7900 2000
@@
 	7500 2100 7500 2150
 $Comp
-L wire_power-rescue:CPC1025NTR-Enigma Q?
+L enigma:CPC1025NTR Q?
 U 1 1 5BED8DC7
 P 9000 2000
@@
 	8600 2100 8600 2150
 $Comp
-L wire_power-rescue:CPC1025NTR-Enigma Q?
+L enigma:CPC1025NTR Q?
 U 1 1 5BED987C
 P 5700 2600
@@
 	5300 2700 5300 2750
 $Comp
-L wire_power-rescue:CPC1025NTR-Enigma Q?
+L enigma:CPC1025NTR Q?
 U 1 1 5BED988D
 P 6800 2600
@@
 	6400 2700 6400 2750
 $Comp
-L wire_power-rescue:CPC1025NTR-Enigma Q?
+L enigma:CPC1025NTR Q?
 U 1 1 5BED989E
 P 7900 2600
@@
 	7500 2700 7500 2750
 $Comp
-L wire_power-rescue:CPC1025NTR-Enigma Q?
+L enigma:CPC1025NTR Q?
 U 1 1 5BED98AF
 P 9000 2600
@@
 	8600 2700 8600 2750
 $Comp
-L wire_power-rescue:CPC1025NTR-Enigma Q?
+L enigma:CPC1025NTR Q?
 U 1 1 5BED98C0
 P 5700 3200
@@
 	5300 3300 5300 3350
 $Comp
-L wire_power-rescue:CPC1025NTR-Enigma Q?
+L enigma:CPC1025NTR Q?
 U 1 1 5BED98D1
 P 6800 3200
@@
 	6400 3300 6400 3350
 $Comp
-L wire_power-rescue:CPC1025NTR-Enigma Q?
+L enigma:CPC1025NTR Q?
 U 1 1 5BED98E2
 P 7900 3200
@@
 	7500 3300 7500 3350
 $Comp
-L wire_power-rescue:CPC1025NTR-Enigma Q?
+L enigma:CPC1025NTR Q?
 U 1 1 5BED98F3
 P 9000 3200
@@
 	8600 3300 8600 3350
 $Comp
-L wire_power-rescue:CPC1025NTR-Enigma Q?
+L enigma:CPC1025NTR Q?
 U 1 1 5BEDAE9E
 P 5700 3850
@@
 	5300 3950 5300 4000
 $Comp
-L wire_power-rescue:CPC1025NTR-Enigma Q?
+L enigma:CPC1025NTR Q?
 U 1 1 5BEDAEAF
 P 6800 3850
@@
 	6400 3950 6400 4000
 $Comp
-L wire_power-rescue:CPC1025NTR-Enigma Q?
+L enigma:CPC1025NTR Q?
 U 1 1 5BEDAEC0
 P 7900 3850
@@
 	7500 3950 7500 4000
 $Comp
-L wire_power-rescue:CPC1025NTR-Enigma Q?
+L enigma:CPC1025NTR Q?
 U 1 1 5BEDAED1
 P 9000 3850
@@
 	8600 3950 8600 4000
 $Comp
-L wire_power-rescue:CPC1025NTR-Enigma Q?
+L enigma:CPC1025NTR Q?
 U 1 1 5BEDAEE2
 P 5700 4450
@@
 	5300 4550 5300 4600
 $Comp
-L wire_power-rescue:CPC1025NTR-Enigma Q?
+L enigma:CPC1025NTR Q?
 U 1 1 5BEDAEF3
 P 6800 4450
@@
 	6400 4550 6400 4600
 $Comp
-L wire_power-rescue:CPC1025NTR-Enigma Q?
+L enigma:CPC1025NTR Q?
 U 1 1 5BEDAF04
 P 7900 4450
@@
 	7500 4550 7500 4600
 $Comp
-L wire_power-rescue:CPC1025NTR-Enigma Q?
+L enigma:CPC1025NTR Q?
 U 1 1 5BEDAF15
 P 9000 4450
@@
 	8600 4550 8600 4600
 $Comp
-L wire_power-rescue:CPC1025NTR-Enigma Q?
+L enigma:CPC1025NTR Q?
 U 1 1 5BEDF896
 P 6800 5050
@@
 	6400 5150 6400 5200
 $Comp
-L wire_power-rescue:CPC1025NTR-Enigma Q?
+L enigma:CPC1025NTR Q?
 U 1 1 5BEDF8A7
 P 7900 5050
@@
 NoConn ~ 1750 2000
 NoConn ~ 1750 1400
+$Comp
+L enigma:Conn_01x26_Male_0 J?
+U 1 1 5BEF48DE
+P 10350 2575
+F 0 "J?" H 10456 3653 50  0000 C CNN
+F 1 "Conn_01x26_Male_0" H 10456 3562 50  0000 C CNN
+F 2 "" H 10350 2575 50  0001 C CNN
+F 3 "" H 10350 2575 50  0001 C CNN
+	1    10350 2575
+	1    0    0    -1
+$EndComp
 $EndSCHEMATC
