File: wire_power/_saved_wire_power.sch (KiCad schematic (older format))
At the start: 61 parts, among them J1 CONN_02X03, J10 Through_hole, J11 Through_hole, J12 Through_hole, J13 Through_hole, J14 Through_hole, J15 Through_hole, J16 Through_hole, J17 Through_hole, J18 Through_hole, J19 Through_hole, J2 CONN_02X03, J20 Through_hole, J21 Through_hole, J22 Through_hole, J23 Through_hole, J24 Through_hole, J25 Through_hole, J26 Through_hole, J27 Through_hole, J28 Through_hole, J29 Through_hole, J4 Through_hole, J5 Through_hole, J6 Through_hole, J7 Through_hole, J8 Through_hole, J9 Through_hole, Q1 CPC1025NTR, Q10 CPC1025NTR, Q11 CPC1025NTR, Q12 CPC1025NTR, Q13 CPC1025NTR, Q14 CPC1025NTR, Q15 CPC1025NTR, Q16 CPC1025NTR, Q17 CPC1025NTR, Q18 CPC1025NTR, Q19 CPC1025NTR, Q2 CPC1025NTR, Q20 CPC1025NTR, Q21 CPC1025NTR, Q22 CPC1025NTR, Q23 CPC1025NTR, Q24 CPC1025NTR, Q25 CPC1025NTR, Q26 CPC1025NTR, Q3 CPC1025NTR, Q4 CPC1025NTR, Q5 CPC1025NTR, Q6 CPC1025NTR, Q7 CPC1025NTR, Q8 CPC1025NTR, Q9 CPC1025NTR, U1 ADG732

Commit message: First pass at wire_power layout UNFINISHED
laid everyhing out in a circle
routed all the MUX ins and outs
Still need to place the input for HOT
Still need to route GND traces
Parts:
- gave numbers to parts that had none: 2
Changed lines of the file:
@@
 NoConn ~ 2850 4250
 $Comp
-L enigma:Through_hole J?
+L enigma:Through_hole J3
 U 1 1 5BFE9737
 P 10550 4275
-F 0 "J?" H 10025 4400 50  0000 C CNN
+F 0 "J3" H 10025 4400 50  0000 C CNN
 F 1 "Through_hole" H 10000 4325 50  0000 C CNN
 F 2 "enigmaprints:thru_hole" H 10550 4275 50  0001 C CNN
@@
 Hot_in
 $Comp
-L enigma:Through_hole J?
+L enigma:Through_hole J30
 U 1 1 5BFF1BB0
 P 10550 4375
-F 0 "J?" H 10025 4500 50  0000 C CNN
+F 0 "J30" H 10025 4500 50  0000 C CNN
 F 1 "Through_hole" H 10000 4425 50  0000 C CNN
 F 2 "enigmaprints:thru_hole" H 10550 4375 50  0001 C CNN
